File: typewriter keyboard.kicad_pcb (KiCad board)
At the start: 2 copper layers, 359.4 x 123.2 mm, 82 parts, among them J1 Conn_01x11_Male, J2 Conn_01x08_Male, J3 Raspberry_Pi_2_3, SW1 SW_Push, SW10 SW_Push, SW11 SW_Push, SW12 SW_Push, SW13 SW_Push, SW14 SW_Push, SW15 SW_Push, SW16 SW_Push, SW17 SW_Push, SW18 SW_Push, SW19 SW_Push, SW2 SW_Push, SW20 SW_Push, SW21 SW_Push, SW22 SW_Push, SW23 SW_Push, SW24 SW_Push, SW25 SW_Push, SW26 SW_Push, SW27 SW_Push, SW28 SW_Push, SW29 SW_Push, SW3 SW_Push, SW30 SW_Push, SW31 SW_Push, SW32 SW_Push, SW33 SW_Push, SW34 SW_Push, SW35 SW_Push, SW36 SW_Push, SW37 SW_Push, SW38 SW_Push, SW39 SW_Push, SW4 SW_Push, SW40 SW_Push, SW41 SW_Push, SW42 SW_Push, SW43 SW_Push, SW44 SW_Push, SW45 SW_Push, SW46 SW_Push, SW47 SW_Push, SW48 SW_Push, SW49 SW_Push, SW5 SW_Push, SW50 SW_Push, SW51 SW_Push, SW52 SW_Push, SW53 SW_Push, SW54 SW_Push, SW55 SW_Push, SW56 SW_Push, SW57 SW_Push, SW58 SW_Push, SW59 SW_Push, SW6 SW_Push, SW60 SW_Push, SW61 SW_Push, SW62 SW_Push, SW63 SW_Push, SW64 SW_Push, SW65 SW_Push, SW66 SW_Push, SW67 SW_Push, SW68 SW_Push, SW69 SW_Push, SW7 SW_Push, SW70 SW_Push, SW8 SW_Push, SW9 SW_Push, U1 CD74HC4067SM, U2 CD74HC4067SM, U3 CD74HC4067SM, U4 CD74HC4067SM, U5 Arduino_Nano

Commit message: Routed PCB, cleaned up schematic
Parts:
- added J4: Conn_01x02_Male, Connector_Wire:SolderWire-0.1sqmm_1x02_P3.6mm_D0.4mm_OD1mm, F.Cu at (349.2, 54.6)
- J3, R1, R2, R3, R4, U1, U2, U3, U4: moved to B.Cu
- SW1, SW10, SW11, SW12, SW13, SW14, SW15, SW17, SW18, SW19, SW2, SW21, SW22, SW23, SW24, SW25, SW26, SW27, SW28, SW29, SW3, SW30, SW31, SW32, SW34, SW35, SW36, SW38, SW39, SW4, SW40, SW41, SW42, SW43, SW44, SW45, SW46, SW47, SW48, SW5, SW50, SW51, SW52, SW54, SW55, SW56, SW57, SW58, SW59, SW6, SW60, SW61, SW62, SW63, SW65, SW7, SW8, SW9: footprint Alps_Only:ALPS-1U -> MX_Alps_Hybrid:MX-1U-NoLED
- SW16: footprint Alps_Only:ALPS-2U -> MX_Alps_Hybrid:MX-2U-NoLED
- SW20, SW33: footprint Alps_Only:ALPS-1.5U -> MX_Alps_Hybrid:MX-1.5U-NoLED
- SW37: footprint Alps_Only:ALPS-1.75U -> MX_Alps_Hybrid:MX-1.75U-NoLED
- SW49, SW53: footprint Alps_Only:ALPS-2.25U -> MX_Alps_Hybrid:MX-2.25U-NoLED
- SW64: footprint Alps_Only:ALPS-2.75U -> MX_Alps_Hybrid:MX-2.75U-NoLED
- SW66, SW67, SW69, SW70: footprint Alps_Only:ALPS-1.25U -> MX_Alps_Hybrid:MX-1.25U-NoLED
- SW68: footprint Alps_Only:ALPS-6.25U -> MX_Alps_Hybrid:MX-6.25U-NoLED
- moved U2 200.7 mm to (62.2, 161.3), turned to 90 degrees
- moved R2 190.3 mm to (321.3, 149.9)
- moved U4 184.2 mm to (321.3, 158.8), turned to 90 degrees
- moved U3 172.3 mm to (334.0, 158.8), turned to 90 degrees
- moved U1 151.8 mm to (185.4, 157.5)
- moved R1 112.1 mm to (196.8, 162.6), turned to 90 degrees
- moved R4 110.6 mm to (351.8, 58.4), turned to -90 degrees
- moved J3 50.8 mm to (363.2, 111.8)
- moved R3 47.5 mm to (351.8, 81.3)
- moved J1 34.3 mm to (157.5, 171.4)
- moved J2 25.4 mm to (54.6, 171.4), turned to 90 degrees
Connections:
- J3 pad 14: GND -> unconnected-(J3-Pad14)
- J3 pad 20: GND -> unconnected-(J3-Pad20)
- J3 pad 25: GND -> unconnected-(J3-Pad25)
- J3 pad 30: GND -> unconnected-(J3-Pad30)
- J3 pad 34: GND -> unconnected-(J3-Pad34)
- J3 pad 39: GND -> unconnected-(J3-Pad39)
- J3 pad 9: GND -> unconnected-(J3-Pad9)
Routing:
- net /Col 8: track 0.00 -> 528.3 mm
- net GND: track 0.00 -> 512.7 mm, vias 0 -> 2
- net /Row 2: track 0.00 -> 473.6 mm
- net /Row 3: track 0.00 -> 472.3 mm, vias 0 -> 1
- net /Col 7: track 0.00 -> 456.4 mm, vias 0 -> 1
- net /Row 8: track 0.00 -> 449.8 mm, vias 0 -> 1
- net /Row 4: track 0.00 -> 449.4 mm, vias 0 -> 1
- net /Row 1: track 0.00 -> 427.5 mm
- net +5V: track 0.00 -> 425.3 mm, vias 0 -> 4
- net /Col 10: track 0.00 -> 411.3 mm, vias 0 -> 1
- net /Row 6: track 0.00 -> 381.6 mm, vias 0 -> 1
- net /Column 11: track 0.00 -> 371.5 mm
- net /Col 9: track 0.00 -> 363.2 mm
- net /Col 2: track 0.00 -> 351.9 mm, vias 0 -> 1
- net /Row 7: track 0.00 -> 350.5 mm
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Other:
- board text added: "+IN"

Commit message: Final changes for order
Parts:
- removed J4: Conn_01x02_Male, Connector_Wire:SolderWire-0.1sqmm_1x02_P3.6mm_D0.4mm_OD1mm
- added +5V1: Conn_01x01_Male, Connector_Wire:SolderWire-0.25sqmm_1x01_D0.65mm_OD1.7mm, F.Cu at (165.1, 55.9)
- added C1: 100u, Capacitor_THT:C_Disc_D3.4mm_W2.1mm_P2.50mm, F.Cu at (191.8, 160.0)
- added C2: 100u, Capacitor_THT:C_Disc_D3.4mm_W2.1mm_P2.50mm, F.Cu at (72.4, 161.3)
- added C3: 100u, Capacitor_THT:C_Disc_D3.4mm_W2.1mm_P2.50mm, F.Cu at (340.4, 154.9)
- added C4: 100u, Capacitor_THT:C_Disc_D3.4mm_W2.1mm_P2.50mm, F.Cu at (327.6, 152.4)
- added G***: LOGO, Arduino:artillect_logo, F.Cu at (39.4, 62.2)
- added G***: LOGO, Arduino:shibui, B.Cu at (213.4, 113.0)
- added GND1: Conn_01x01_Male, Connector_Wire:SolderWire-0.25sqmm_1x01_D0.65mm_OD1.7mm, F.Cu at (299.7, 55.9)
- added R5: 330, Resistor_THT:R_Axial_DIN0207_L6.3mm_D2.5mm_P10.16mm_Horizontal, B.Cu at (365.8, 124.5)
- R4: value 660 -> 330
- moved R4 80.7 mm to (361.9, 138.4), turned to 90 degrees
- moved R3 68.7 mm to (365.8, 148.6)
Connections:
- R4 pad 2: Net-(J3-Pad10) -> Net-(R4-Pad2)
- U5 pad 27: unconnected-(U5-Pad27) -> +5V
- U5 pad 30: +5V -> unconnected-(U5-Pad30)
Routing:
- net +5V: track 425.3 -> 623.7 mm, vias 4 -> 3
- net Net-(R3-Pad1): track 96.8 -> 28.1 mm
- net Net-(J3-Pad10): track 11.4 -> 76.3 mm
- net GND: track 512.7 -> 533.9 mm, vias 2 -> 4
- net /Col 2: track 351.9 -> 368.7 mm
- net /KB SIG: track 73.8 -> 84.3 mm, vias 0 -> 1
- net /Col 3: track 327.9 -> 337.2 mm
- net /Col 8: track 528.3 -> 536.6 mm
- net Net-(R4-Pad2): track 0.00 -> 5.39 mm
- net /Col 4: track 298.2 -> 303.2 mm, vias 1 -> 3
- net /Row 1: track 427.5 -> 431.5 mm
- net /Col 7: track 456.4 -> 460.4 mm, vias 1 -> 2
- net /Column 11: track 371.5 -> 375.4 mm
- net /Col 10: track 411.3 -> 415.1 mm
- net /Row 2: track 473.6 -> 476.9 mm
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- added copper zone on B.Cu, net GND
Other:
- board text added: "Brother AX-25 Teletype Conversion Board Rev 1.0 9 September 2022 Artillect"
- board text removed: "+IN"
